Commit message: Made the main URDF File
Finished exporting the last of the parts.

File: Arm 2024-2025/Arm URDF/urdf/Arm URDF.urdf (robot description, URDF)
Before this commit: robot Arm URDF, 3 links, 2 joints
Links:
- removed link link_1
- removed link shoulder_base
- added link a1_shoulder_base, mass 0.742438926040346; collision mesh filename=package://Arm URDF/meshes/a1_shoulder_base.STL; visual mesh filename=package://Arm URDF/meshes/a1_shoulder_base.STL
- added link a2_link_1, mass 1.94678380458644; collision mesh filename=package://Arm URDF/meshes/a2_link_1.STL; visual mesh filename=package://Arm URDF/meshes/a2_link_1.STL
- added link a3_axis4_housing, mass 0.258864677478161; collision mesh filename=package://Arm URDF/meshes/a3_axis4_housing.STL; visual mesh filename=package://Arm URDF/meshes/a3_axis4_housing.STL
- added link a4_link2, mass 1.31628289409256; collision mesh filename=package://Arm URDF/meshes/a4_link2.STL; visual mesh filename=package://Arm URDF/meshes/a4_link2.STL
- added link a5_internal_upright, mass 0.155027470866593; collision mesh filename=package://Arm URDF/meshes/a5_internal_upright.STL; visual mesh filename=package://Arm URDF/meshes/a5_internal_upright.STL
- added link a6_EE_holder, mass 0.268420822776766; collision mesh filename=package://Arm URDF/meshes/a6_EE_holder.STL; visual mesh filename=package://Arm URDF/meshes/a6_EE_holder.STL
Joints:
- added joint a4_rotation: type revolute, parent a3_axis4_housing, child a4_link2, origin xyz=0.0451078368209206 0.205024453664939 0.223589169838865 rpy=-1.5707963267949 -0.828683805160042 1.5707963267949, axis -1 0 0, limit lower=-1.57 upper=1.57 effort=0 velocity=0
- added joint a5_rotation: type revolute, parent a4_link2, child a5_internal_upright, origin xyz=0.31694 0 0.024001 rpy=0.74211 1.5708 0, axis 1 0 0, limit lower=-3.14 upper=3.14 effort=0 velocity=0
- added joint a6_rotation: type continuous, parent a5_internal_upright, child a6_EE_holder, origin xyz=0.024 0.031992 0.030931 rpy=-1.5708 -0.76854 1.5708, axis -1 0 0, limit lower=0 upper=0 effort=0 velocity=0
- added joint link1_link2: type revolute, parent a2_link_1, child a3_axis4_housing, origin xyz=-0.50000048929394 0 -0.0677177243260161 rpy=0 1.5707963267949 0, axis -1 0 0, limit lower=0 upper=3.14 effort=0 velocity=0
- joint link_1_joint: axis 0 0 -1 -> 0 0 1; child link_1 -> a2_link_1; limit lower=0 upper=3.14 effort=0 velocity=0 -> lower=-3.14 upper=0 effort=0 velocity=0; origin xyz=-0.00275 -0.045 0.075 rpy=0 -1.5708 0 -> xyz=0.00282500000000498 -0.0450000000000385 0.074999999999904 rpy=1.5707963267949 0 -1.5707963267949; parent shoulder_base -> a1_shoulder_base
- joint shoulder_joint: child shoulder_base -> a1_shoulder_base; origin xyz=0.102 0.2 0.03775 rpy=0 0 -3.1416 -> xyz=0.102000000000005 0.199999999999999 0.0377499999999958 rpy=0 0 -3.14159265358979
